File: CESP.sch (KiCad schematic (older format))
At the start: 5 parts

Commit message: Not really a solder practice any more
Parts:
- removed U?: LTC1594CS, TSSOP14, symbol LTC1594CS
- removed U?: TL074, TSSOP14, symbol TL074
- removed U? (x3): TL074, symbol TL074
- added CN1: BNC, BNC-RIGHT-ANGLE-PLASTIC, symbol BNC
- added J1: SIL4, SIL-4, symbol SIL4
- added J2: SIL4, symbol SIL4
- added VR1: 10R, RV-BLUE-PLASTIC, symbol VR
- added VR2: 200R, RV-BLUE-PLASTIC, symbol VR
Connections:
- net labels added: GND
- wire segments 0 -> 8
Other:
- note removed: "NOTE: THIS IS JUST A TEST BOARD\nREMOVE ALL COMPONENTS AND CREATE YOUR OWN\nINCLUDE SCHEMATIC HOOKUPS/NETLIST"
Changed lines of the file:
@@
-EESchema Schematic File Version 2  date 1/24/2014 12:04:40 AM
+EESchema Schematic File Version 2
+LIBS:custom
 LIBS:power
 LIBS:device
@@
 Sheet 1 1
 Title ""
-Date "24 jan 2014"
+Date "26 jan 2014"
 Rev ""
 Comp ""
@@
 $EndDescr
 $Comp
-L LTC1594CS U?
-U 1 1 52E1F38F
-P 3750 3300
-F 0 "U?" H 3750 3950 60  0000 C CNN
-F 1 "LTC1594CS" H 3750 2650 60  0000 C CNN
-F 2 "TSSOP14" H 3750 3300 60  0000 C CNN
-F 3 "" H 3750 3300 60  0000 C CNN
-	1    3750 3300
+L VR VR2
+U 1 1 52E4AFFE
+P 3200 1850
+F 0 "VR2" V 3260 1804 40  0000 C TNN
+F 1 "200R" V 3200 1850 40  0000 C CNN
+F 2 "RV-BLUE-PLASTIC" H 3200 1850 60  0001 C CNN
+F 3 "~" H 3200 1850 60  0000 C CNN
+	1    3200 1850
+	0    1    1    0
+$EndComp
+$Comp
+L VR VR1
+U 1 1 52E4B00B
+P 2700 1850
+F 0 "VR1" V 2760 1804 40  0000 C TNN
+F 1 "10R" V 2700 1850 40  0000 C CNN
+F 2 "RV-BLUE-PLASTIC" H 2700 1850 60  0001 C CNN
+F 3 "~" H 2700 1850 60  0000 C CNN
+	1    2700 1850
+	0    1    1    0
+$EndComp
+$Comp
+L BNC CN1
+U 1 1 52E4F0C4
+P 2550 1600
+F 0 "CN1" H 2560 1720 60  0000 C CNN
+F 1 "BNC" V 2660 1540 40  0000 C CNN
+F 2 "BNC-RIGHT-ANGLE-PLASTIC" H 2550 1600 60  0001 C CNN
+F 3 "~" H 2550 1600 60  0000 C CNN
+	1    2550 1600
+	0    -1   1    0
+$EndComp
+$Comp
+L SIL4 J1
+U 1 1 52E50F02
+P 2600 900
+F 0 "J1" H 2600 1150 70  0000 C CNN
+F 1 "SIL4" V 2620 900 70  0000 C CNN
+F 2 "SIL-4" H 2600 900 60  0001 C CNN
+F 3 "" H 2600 900 60  0000 C CNN
+	1    2600 900
+	0    -1   -1   0
+$EndComp
+Text GLabel 2750 1600 2    60   Input ~ 0
+GND
+Text GLabel 3450 1850 2    60   Input ~ 0
+GND
+Text GLabel 2650 1250 3    60   Input ~ 0
+GND
+Wire Wire Line
+	2450 1250 2450 1850
+Wire Wire Line
+	2550 1250 2550 1450
+$Comp
+L SIL4 J2
+U 1 1 52E539B0
+P 3350 1000
+F 0 "J2" H 3350 1250 70  0000 C CNN
+F 1 "SIL4" V 3370 1000 70  0000 C CNN
+F 2 "" H 3350 1000 60  0000 C CNN
+F 3 "" H 3350 1000 60  0000 C CNN
+	1    3350 1000
 	1    0    0    -1
 $EndComp
-$Comp
-L TL074 U?
-U 1 1 52E1F3CD
-P 7150 2150
-F 0 "U?" H 7200 2350 60  0000 C CNN
-F 1 "TL074" H 7300 1950 50  0000 C CNN
-F 2 "TSSOP14" H 7150 2150 60  0000 C CNN
-F 3 "" H 7150 2150 60  0000 C CNN
-	1    7150 2150
-	1    0    0    -1
-$EndComp
-$Comp
-L TL074 U?
-U 2 1 52E1F3DA
-P 7200 3500
-F 0 "U?" H 7250 3700 60  0000 C CNN
-F 1 "TL074" H 7350 3300 50  0000 C CNN
-F 2 "" H 7200 3500 60  0000 C CNN
-F 3 "" H 7200 3500 60  0000 C CNN
-	2    7200 3500
-	1    0    0    -1
-$EndComp
-$Comp
-L TL074 U?
-U 1 1 52E1F3E5
-P 8600 3500
-F 0 "U?" H 8650 3700 60  0000 C CNN
-F 1 "TL074" H 8750 3300 50  0000 C CNN
-F 2 "" H 8600 3500 60  0000 C CNN
-F 3 "" H 8600 3500 60  0000 C CNN
-	1    8600 3500
-	1    0    0    -1
-$EndComp
-$Comp
-L TL074 U?
-U 1 1 52E1F3EB
-P 8550 2100
-F 0 "U?" H 8600 2300 60  0000 C CNN
-F 1 "TL074" H 8700 1900 50  0000 C CNN
-F 2 "" H 8550 2100 60  0000 C CNN
-F 3 "" H 8550 2100 60  0000 C CNN
-	1    8550 2100
-	1    0    0    -1
-$EndComp
-Text Notes 4450 4650 0    80   ~ 0
-NOTE: THIS IS JUST A TEST BOARD\nREMOVE ALL COMPONENTS AND CREATE YOUR OWN\nINCLUDE SCHEMATIC HOOKUPS/NETLIST
+Wire Wire Line
+	2550 1450 2900 1450
+Wire Wire Line
+	2900 1450 2900 950
+Wire Wire Line
+	2900 950  3000 950
+Wire Wire Line
+	3000 850  2850 850
+Wire Wire Line
+	2850 850  2850 1250
+Wire Wire Line
+	2850 1250 2750 1250
 $EndSCHEMATC
